Commit message: Details un README, re-importing quadruped

File: quadruped/robot.urdf (robot description, URDF)
Before this commit: robot onshape, 15 links, 14 joints
Joints:
- joint leg2_c: origin xyz=-0.063 -1.53523e-15 4.28477e-16 rpy=1.5708 1.64389e-15 1.5708 -> xyz=-0.063 -1.53176e-15 7.45931e-17 rpy=1.5708 1.64389e-15 1.5708
- joint leg3_c: origin xyz=-0.063 -1.37217e-15 -2.77556e-17 rpy=1.5708 1.28111e-16 1.5708 -> xyz=-0.063 -1.37217e-15 -5.89806e-17 rpy=1.5708 1.28111e-16 1.5708
- joint tip_frame: origin xyz=0.0025 0.015 -0.1005 rpy=4.29183e-32 1.5708 0 -> xyz=0.0025 0.015 -0.1005 rpy=1.41526e-31 1.5708 0

Commit message: Merging STLs in quadruped

File: quadruped/robot.urdf (robot description, URDF)
Before this commit: robot onshape, 15 links, 14 joints
Links:
- link body_1: geometry collision box size=0.02 0.03 0.022; collision box size=0.02 0.03 0.022
- link doubleu_1: geometry collision box size=0.02 0.03 0.002; collision box size=0.02 0.03 0.002
- link doubleu_2: geometry collision box size=0.02 0.03 0.002; collision box size=0.02 0.03 0.002
- link doubleu_3: geometry collision box size=0.02 0.03 0.002; collision box size=0.02 0.03 0.002
- link doubleu_4: geometry collision box size=0.02 0.03 0.002; collision box size=0.02 0.03 0.002
- link leg_1: geometry collision box size=0.02 0.002 0.09; collision box size=0.02 0.002 0.09
- link leg_2: geometry collision box size=0.02 0.002 0.09; collision box size=0.02 0.002 0.09
- link leg_3: geometry collision box size=0.02 0.002 0.09; collision box size=0.02 0.002 0.09
- link leg_4: geometry collision box size=0.02 0.002 0.09; collision box size=0.02 0.002 0.09
- link platesblock_1: geometry collision box size=0.02 0.03 0.022; collision box size=0.02 0.03 0.022
- link platesblock_2: geometry collision box size=0.02 0.03 0.022; collision box size=0.02 0.03 0.022
- link platesblock_3: geometry collision box size=0.02 0.03 0.022; collision box size=0.02 0.03 0.022
- link platesblock_4: geometry collision box size=0.02 0.03 0.022; collision box size=0.02 0.03 0.022
