Commit message: useFixedLinks

File: field/robot.urdf (robot description, URDF)
Before this commit: robot onshape, 12 links, 11 joints
Links:
- removed link goalsally_1
- removed link goalsallyback_1
- removed link goalsopponent_1
- removed link goalsopponentback_1
- removed link lines_1
- removed link penaltyally_1
- removed link penaltyopponent_1
- removed link table2_1
- removed link table3_1
- removed link table4_1
- removed link table_1
- added link field_1_1, mass 0; visual mesh filename=package://table4.stl
- added link field_1_10, mass 0; visual mesh filename=package://field.stl
- added link field_1_11, mass 0; visual mesh filename=package://penaltyally.stl
- added link field_1_12, mass 0; visual mesh filename=package://lines.stl
- added link field_1_2, mass 0; visual mesh filename=package://penaltyopponent.stl
- added link field_1_3, mass 0; visual mesh filename=package://goalsally.stl
- added link field_1_4, mass 0; visual mesh filename=package://table2.stl
- added link field_1_5, mass 0; visual mesh filename=package://table3.stl
- added link field_1_6, mass 0; visual mesh filename=package://goalsopponent.stl
- added link field_1_7, mass 0; visual mesh filename=package://table.stl
- added link field_1_8, mass 0; visual mesh filename=package://goalsallyback.stl
- added link field_1_9, mass 0; visual mesh filename=package://goalsopponentback.stl
- link field_1: geometry collision mesh filename=package://field.stl; collision mesh filename=package://goalsally.stl
Joints:
- removed joint 0310c999-4296-4db8-9f39-83df45833534
- removed joint 214b5820-0449-45be-a81b-332eed3c51f5
- removed joint 4f383524-a167-4cbd-a1bc-ad6fa655fc4b
- removed joint 6a2a839b-5e2c-4478-a103-f1c1f69f211d
- removed joint 9aa094e6-9425-42d6-bb35-2fb61ac98efc
- removed joint c16b3023-a020-4846-9529-9f5a85b979a0
- removed joint ccd0940d-cd18-4f6a-8444-c234a5fc23ea
- removed joint d389819a-6b39-4795-bd4e-0864f09296de
- removed joint db882b0d-06d5-4f69-ba80-12af02025efd
- removed joint e8f8e501-26f0-40bc-9401-a50023d60e52
- removed joint fda29d22-884a-4018-923e-5919f2ec4442
- added joint field_1_10_fixing: type fixed, parent field_1, child field_1_10, origin xyz=0 0 0 rpy=0 -0 0, axis 0 0 1, limit effort=1 velocity=20
- added joint field_1_11_fixing: type fixed, parent field_1, child field_1_11, origin xyz=0 0 0 rpy=0 -0 0, axis 0 0 1, limit effort=1 velocity=20
- added joint field_1_12_fixing: type fixed, parent field_1, child field_1_12, origin xyz=0 0 0 rpy=0 -0 0, axis 0 0 1, limit effort=1 velocity=20
- added joint field_1_1_fixing: type fixed, parent field_1, child field_1_1, origin xyz=0 0 0 rpy=0 -0 0, axis 0 0 1, limit effort=1 velocity=20
- added joint field_1_2_fixing: type fixed, parent field_1, child field_1_2, origin xyz=0 0 0 rpy=0 -0 0, axis 0 0 1, limit effort=1 velocity=20
- added joint field_1_3_fixing: type fixed, parent field_1, child field_1_3, origin xyz=0 0 0 rpy=0 -0 0, axis 0 0 1, limit effort=1 velocity=20
- added joint field_1_4_fixing: type fixed, parent field_1, child field_1_4, origin xyz=0 0 0 rpy=0 -0 0, axis 0 0 1, limit effort=1 velocity=20
- added joint field_1_5_fixing: type fixed, parent field_1, child field_1_5, origin xyz=0 0 0 rpy=0 -0 0, axis 0 0 1, limit effort=1 velocity=20
- added joint field_1_6_fixing: type fixed, parent field_1, child field_1_6, origin xyz=0 0 0 rpy=0 -0 0, axis 0 0 1, limit effort=1 velocity=20
- added joint field_1_7_fixing: type fixed, parent field_1, child field_1_7, origin xyz=0 0 0 rpy=0 -0 0, axis 0 0 1, limit effort=1 velocity=20
- added joint field_1_8_fixing: type fixed, parent field_1, child field_1_8, origin xyz=0 0 0 rpy=0 -0 0, axis 0 0 1, limit effort=1 velocity=20
- added joint field_1_9_fixing: type fixed, parent field_1, child field_1_9, origin xyz=0 0 0 rpy=0 -0 0, axis 0 0 1, limit effort=1 velocity=20
