Commit message: Using _speed in 2wheels dof to make them speed controlled instead

File: 2wheels/robot.urdf (robot description, URDF)
Before this commit: robot onshape, 3 links, 2 joints
Links:
- link wheel_1: geometry collision mesh filename=package://wheel.stl; visual mesh filename=package://wheel.stl
- link wheel_2: geometry collision mesh filename=package://wheel.stl; visual mesh filename=package://wheel.stl
Joints:
- removed joint wheel1
- removed joint wheel2
- added joint wheel1_speed: type revolute, parent body_1, child wheel_1, origin xyz=-0.02 0.0325 0.025 rpy=0 -0 0, axis -1 0 0, limit effort=1 velocity=20
- added joint wheel2_speed: type revolute, parent body_1, child wheel_2, origin xyz=0.095 0.0325 0.025 rpy=0 -0 0, axis 1 0 0, limit effort=1 velocity=20

Commit message: Example of _inv and _speed explained

File: 2wheels/robot.urdf (robot description, URDF)
Before this commit: robot onshape, 3 links, 2 joints
Joints:
- joint wheel2_speed: axis 1 0 0 -> -1 -0 -0

Commit message: Updating 2wheel example with latest version

File: 2wheels/robot.urdf (robot description, URDF)
Before this commit: robot onshape, 3 links, 2 joints
Links:
- removed link body_1
- removed link wheel_1
- added link body, mass 2.23874; collision mesh filename=package://body.stl; visual mesh filename=package://body.stl
- added link wheel, mass 0.335419; collision mesh filename=package://wheel.stl; visual mesh filename=package://wheel.stl
Joints:
- joint wheel1_speed: axis -1 0 0 -> 0 0 1; child wheel_1 -> wheel; limit effort=1 velocity=20 -> effort=10 velocity=10; origin xyz=-0.02 0.0325 0.025 rpy=0 -0 0 -> xyz=-0.02 0.0325 0.025 rpy=-1.5708 -0 1.5708; parent body_1 -> body; type revolute -> continuous
- joint wheel2_speed: axis -1 -0 -0 -> 0 0 1; limit effort=1 velocity=20 -> effort=10 velocity=10; origin xyz=0.095 0.0325 0.025 rpy=0 -0 0 -> xyz=0.095 0.0325 0.025 rpy=-1.5708 -0 1.5708; parent body_1 -> body; type revolute -> continuous
