Commit message: Updating 2wheel example

File: 2wheels_urdf/robot.urdf (robot description, URDF)
Before this commit: robot 2wheels_urdf, 3 links, 2 joints
Links:
- link body: geometry collision mesh filename=package://assets/body.stl; visual mesh filename=package://assets/body.stl
- link wheel: geometry collision mesh filename=package://assets/wheel.stl; visual mesh filename=package://assets/wheel.stl
- link wheel_2: geometry collision mesh filename=package://assets/wheel.stl; visual mesh filename=package://assets/wheel.stl
