Commit message: Updating adjustable height arm example

File: adjustable_height_arm_urdf/robot.urdf (robot description, URDF)
Before this commit: robot adjustable_height_arm_urdf, 6 links, 5 joints
Links:
- link base: mass 0.39382 -> 0; geometry visual mesh filename=package://assets/base.stl
- link part1: geometry visual mesh filename=package://assets/part1.stl
- link part2: geometry visual mesh filename=package://assets/part2.stl
- link part3: geometry visual mesh filename=package://assets/part3.stl
- link part4: geometry visual mesh filename=package://assets/part4.stl
