Commit message: Updating omnidirectional example

File: omnidirectional_urdf/robot.urdf (robot description, URDF)
Before this commit: robot omnidirectional_urdf, 65 links, 64 joints
Links:
- link body_2: geometry visual mesh filename=package://assets/motor.stl; visual mesh filename=package://assets/motor.stl
- link passivewheel: geometry collision cylinder length=0.003 radius=0.006; visual mesh filename=package://assets/passivewheel.stl
- link passivewheel_10: geometry collision cylinder length=0.003 radius=0.006; visual mesh filename=package://assets/passivewheel.stl
- link passivewheel_11: geometry collision cylinder length=0.003 radius=0.006; visual mesh filename=package://assets/passivewheel.stl
- link passivewheel_12: geometry collision cylinder length=0.003 radius=0.006; visual mesh filename=package://assets/passivewheel.stl
- link passivewheel_13: geometry collision cylinder length=0.003 radius=0.006; visual mesh filename=package://assets/passivewheel.stl
- link passivewheel_14: geometry collision cylinder length=0.003 radius=0.006; visual mesh filename=package://assets/passivewheel.stl
- link passivewheel_15: geometry collision cylinder length=0.003 radius=0.006; visual mesh filename=package://assets/passivewheel.stl
- link passivewheel_16: geometry collision cylinder length=0.003 radius=0.006; visual mesh filename=package://assets/passivewheel.stl
- link passivewheel_17: geometry collision cylinder length=0.003 radius=0.006; visual mesh filename=package://assets/passivewheel.stl
- link passivewheel_18: geometry collision cylinder length=0.003 radius=0.006; visual mesh filename=package://assets/passivewheel.stl
- link passivewheel_19: geometry collision cylinder length=0.003 radius=0.006; visual mesh filename=package://assets/passivewheel.stl
- link passivewheel_2: geometry collision cylinder length=0.003 radius=0.006; visual mesh filename=package://assets/passivewheel.stl
- link passivewheel_20: geometry collision cylinder length=0.003 radius=0.006; visual mesh filename=package://assets/passivewheel.stl
- link passivewheel_21: geometry collision cylinder length=0.003 radius=0.006; visual mesh filename=package://assets/passivewheel.stl
- link passivewheel_22: geometry collision cylinder length=0.003 radius=0.006; visual mesh filename=package://assets/passivewheel.stl
- link passivewheel_23: geometry collision cylinder length=0.003 radius=0.006; visual mesh filename=package://assets/passivewheel.stl
- link passivewheel_24: geometry collision cylinder length=0.003 radius=0.006; visual mesh filename=package://assets/passivewheel.stl
- link passivewheel_25: geometry collision cylinder length=0.003 radius=0.006; visual mesh filename=package://assets/passivewheel.stl
- link passivewheel_26: geometry collision cylinder length=0.003 radius=0.006; visual mesh filename=package://assets/passivewheel.stl
- link passivewheel_27: geometry collision cylinder length=0.003 radius=0.006; visual mesh filename=package://assets/passivewheel.stl
- link passivewheel_28: geometry collision cylinder length=0.003 radius=0.006; visual mesh filename=package://assets/passivewheel.stl
- link passivewheel_29: geometry collision cylinder length=0.003 radius=0.006; visual mesh filename=package://assets/passivewheel.stl
- link passivewheel_3: geometry collision cylinder length=0.003 radius=0.006; visual mesh filename=package://assets/passivewheel.stl
- link passivewheel_30: geometry collision cylinder length=0.003 radius=0.006; visual mesh filename=package://assets/passivewheel.stl
- link passivewheel_31: geometry collision cylinder length=0.003 radius=0.006; visual mesh filename=package://assets/passivewheel.stl
- link passivewheel_32: geometry collision cylinder length=0.003 radius=0.006; visual mesh filename=package://assets/passivewheel.stl
- link passivewheel_33: geometry collision cylinder length=0.003 radius=0.006; visual mesh filename=package://assets/passivewheel.stl
- link passivewheel_34: geometry collision cylinder length=0.003 radius=0.006; visual mesh filename=package://assets/passivewheel.stl
- link passivewheel_35: geometry collision cylinder length=0.003 radius=0.006; visual mesh filename=package://assets/passivewheel.stl
- link passivewheel_36: geometry collision cylinder length=0.003 radius=0.006; visual mesh filename=package://assets/passivewheel.stl
- link passivewheel_37: geometry collision cylinder length=0.003 radius=0.006; visual mesh filename=package://assets/passivewheel.stl
- link passivewheel_38: geometry collision cylinder length=0.003 radius=0.006; visual mesh filename=package://assets/passivewheel.stl
- link passivewheel_39: geometry collision cylinder length=0.003 radius=0.006; visual mesh filename=package://assets/passivewheel.stl
- link passivewheel_4: geometry collision cylinder length=0.003 radius=0.006; visual mesh filename=package://assets/passivewheel.stl
- link passivewheel_40: geometry collision cylinder length=0.003 radius=0.006; visual mesh filename=package://assets/passivewheel.stl
- link passivewheel_41: geometry collision cylinder length=0.003 radius=0.006; visual mesh filename=package://assets/passivewheel.stl
- link passivewheel_42: geometry collision cylinder length=0.003 radius=0.006; visual mesh filename=package://assets/passivewheel.stl
- link passivewheel_43: geometry collision cylinder length=0.003 radius=0.006; visual mesh filename=package://assets/passivewheel.stl
- link passivewheel_44: geometry collision cylinder length=0.003 radius=0.006; visual mesh filename=package://assets/passivewheel.stl
- link passivewheel_45: geometry collision cylinder length=0.003 radius=0.006; visual mesh filename=package://assets/passivewheel.stl
- link passivewheel_46: geometry collision cylinder length=0.003 radius=0.006; visual mesh filename=package://assets/passivewheel.stl
- link passivewheel_47: geometry collision cylinder length=0.003 radius=0.006; visual mesh filename=package://assets/passivewheel.stl
- link passivewheel_48: geometry collision cylinder length=0.003 radius=0.006; visual mesh filename=package://assets/passivewheel.stl
- link passivewheel_49: geometry collision cylinder length=0.003 radius=0.006; visual mesh filename=package://assets/passivewheel.stl
- link passivewheel_5: geometry collision cylinder length=0.003 radius=0.006; visual mesh filename=package://assets/passivewheel.stl
- link passivewheel_50: geometry collision cylinder length=0.003 radius=0.006; visual mesh filename=package://assets/passivewheel.stl
- link passivewheel_51: geometry collision cylinder length=0.003 radius=0.006; visual mesh filename=package://assets/passivewheel.stl
- link passivewheel_52: geometry collision cylinder length=0.003 radius=0.006; visual mesh filename=package://assets/passivewheel.stl
- link passivewheel_53: geometry collision cylinder length=0.003 radius=0.006; visual mesh filename=package://assets/passivewheel.stl
- link passivewheel_54: geometry collision cylinder length=0.003 radius=0.006; visual mesh filename=package://assets/passivewheel.stl
- link passivewheel_55: geometry collision cylinder length=0.003 radius=0.006; visual mesh filename=package://assets/passivewheel.stl
- link passivewheel_56: geometry collision cylinder length=0.003 radius=0.006; visual mesh filename=package://assets/passivewheel.stl
- link passivewheel_57: geometry collision cylinder length=0.003 radius=0.006; visual mesh filename=package://assets/passivewheel.stl
- link passivewheel_58: geometry collision cylinder length=0.003 radius=0.006; visual mesh filename=package://assets/passivewheel.stl
- link passivewheel_59: geometry collision cylinder length=0.003 radius=0.006; visual mesh filename=package://assets/passivewheel.stl
- link passivewheel_6: geometry collision cylinder length=0.003 radius=0.006; visual mesh filename=package://assets/passivewheel.stl
- link passivewheel_60: geometry collision cylinder length=0.003 radius=0.006; visual mesh filename=package://assets/passivewheel.stl
- link passivewheel_7: geometry collision cylinder length=0.003 radius=0.006; visual mesh filename=package://assets/passivewheel.stl
- link passivewheel_8: geometry collision cylinder length=0.003 radius=0.006; visual mesh filename=package://assets/passivewheel.stl
- link passivewheel_9: geometry collision cylinder length=0.003 radius=0.006; visual mesh filename=package://assets/passivewheel.stl
- link wheel: geometry visual mesh filename=package://assets/wheel.stl
- link wheel_2: geometry visual mesh filename=package://assets/wheel.stl
- link wheel_3: geometry visual mesh filename=package://assets/wheel.stl
