Commit message: Updating quadruped example

File: quadruped_urdf/robot.urdf (robot description, URDF)
Before this commit: robot quadruped_urdf, 14 links, 13 joints
Links:
- link body: geometry collision box size=0.02 0.03 0.022; collision box size=0.02 0.03 0.022
- link doubleu: geometry collision box size=0.02 0.03 0.002; collision box size=0.02 0.03 0.002
- link doubleu_2: geometry collision box size=0.02 0.03 0.002; collision box size=0.02 0.03 0.002
- link doubleu_3: geometry collision box size=0.02 0.03 0.002; collision box size=0.02 0.03 0.002
- link doubleu_4: geometry collision box size=0.02 0.03 0.002; collision box size=0.02 0.03 0.002
- link leg: geometry collision box size=0.02 0.002 0.09; collision box size=0.02 0.002 0.09
- link leg_2: geometry collision box size=0.02 0.002 0.09; collision box size=0.02 0.002 0.09
- link leg_3: geometry collision box size=0.02 0.002 0.09; collision box size=0.02 0.002 0.09
- link leg_4: geometry collision box size=0.02 0.002 0.09; collision box size=0.02 0.002 0.09
- link platesblock: geometry collision box size=0.02 0.03 0.022; collision box size=0.02 0.03 0.022
- link platesblock_2: geometry collision box size=0.02 0.03 0.022; collision box size=0.02 0.03 0.022
- link platesblock_3: geometry collision box size=0.02 0.03 0.022; collision box size=0.02 0.03 0.022
- link platesblock_4: geometry collision box size=0.02 0.03 0.022; collision box size=0.02 0.03 0.022
