Commit message: Updating sigmaban example

File: sigmaban2019_urdf/robot.urdf (robot description, URDF)
Before this commit: robot sigmaban2019_urdf, 27 links, 26 joints
Links:
- link head: geometry collision box size=0.008 0.05 0.003; collision box size=0.008 0.05 0.003
- link left_foot_cleat_front_right: geometry collision box size=0.01 0.09 0.01; collision box size=0.025 0.044 0.003
- link left_humerus: geometry collision box size=0.003 0.07 0.03; collision box size=0.029 0.05 0.04
- link left_knee: geometry collision box size=0.03 0.055 0.04; collision box size=0.04 0.09 0.003
- link left_radius: geometry collision box size=0.003 0.085 0.03; collision box size=0.029 0.05 0.04
- link mx106_block: geometry collision box size=0.03 0.055 0.04; collision box size=0.03 0.055 0.04
- link mx106_block_2: geometry collision box size=0.03 0.055 0.04; collision box size=0.03 0.055 0.04
- link mx106_block_mir: geometry collision box size=0.03 0.055 0.04; collision box size=0.03 0.055 0.04
- link mx106_block_mir_2: geometry collision box size=0.03 0.055 0.04; collision box size=0.03 0.055 0.04
- link right_foot_cleat_back_left: geometry collision box size=0.01 0.09 0.01; collision box size=0.025 0.044 0.003
- link right_humerus: geometry collision box size=0.003 0.07 0.03; collision box size=0.029 0.05 0.04
- link right_knee: geometry collision box size=0.03 0.055 0.04; collision box size=0.04 0.09 0.003
- link right_radius: geometry collision box size=0.003 0.085 0.03; collision box size=0.029 0.05 0.04
- link tibia: geometry collision box size=0.03 0.165 0.003; collision box size=0.03 0.165 0.003
- link tibia_2: geometry collision box size=0.03 0.165 0.003; collision box size=0.03 0.165 0.003
- link tronc: geometry collision box size=0.01 0.035 0.003; collision box size=0.01 0.035 0.003
- link u_block: geometry collision box size=0.025 0.044 0.003; collision box size=0.027 0.042 0.003
- link u_block_2: geometry collision box size=0.025 0.044 0.003; collision box size=0.027 0.042 0.003
- link u_neck: geometry collision box size=0.025 0.044 0.003; collision box size=0.025 0.044 0.003
- link u_shoulder: geometry visual mesh filename=package://assets/merged/u_shoulder.stl
- link u_shoulder_2: geometry visual mesh filename=package://assets/merged/u_shoulder_2.stl
Joints:
- joint left_shoulder_pitch: origin xyz=0.0735 -0.032127 0.1609 rpy=-1.5708 -4.55145e-13 -1.5708 -> xyz=0.0735 -0.032127 0.1609 rpy=-1.5708 -5.08852e-16 -1.5708
- joint left_shoulder_roll: origin xyz=0.0225 0.03 0.035 rpy=-3.14159 -1.5708 0 -> xyz=0.0225 0.03 0.035 rpy=3.14159 -1.5708 0
