Commit message: Details

File: field_urdf/robot.urdf (robot description, URDF)
Before this commit: robot onshape-to-robot-examples, 13 links, 12 joints
Links:
- removed link field_field
- removed link field_goalsally
- removed link field_goalsallyback
- removed link field_goalsopponent
- removed link field_goalsopponentback
- removed link field_lines
- removed link field_penaltyally
- removed link field_penaltyopponent
- removed link field_table
- removed link field_table2
- removed link field_table3
- removed link field_table4
- added link base_link, mass 0
- added link goalsally, mass 0; collision mesh filename=package://goalsally.stl; visual mesh filename=package://goalsally.stl
- added link goalsallyback, mass 0; collision mesh filename=package://goalsallyback.stl; visual mesh filename=package://goalsallyback.stl
- added link goalsopponent, mass 0; collision mesh filename=package://goalsopponent.stl; visual mesh filename=package://goalsopponent.stl
- added link goalsopponentback, mass 0; collision mesh filename=package://goalsopponentback.stl; visual mesh filename=package://goalsopponentback.stl
- added link lines, mass 0; collision mesh filename=package://lines.stl; visual mesh filename=package://lines.stl
- added link penaltyally, mass 0; collision mesh filename=package://penaltyally.stl; visual mesh filename=package://penaltyally.stl
- added link penaltyopponent, mass 0; collision mesh filename=package://penaltyopponent.stl; visual mesh filename=package://penaltyopponent.stl
- added link table, mass 0; collision mesh filename=package://table.stl; visual mesh filename=package://table.stl
- added link table2, mass 0; collision mesh filename=package://table2.stl; visual mesh filename=package://table2.stl
- added link table3, mass 0; collision mesh filename=package://table3.stl; visual mesh filename=package://table3.stl
- added link table4, mass 0; collision mesh filename=package://table4.stl; visual mesh filename=package://table4.stl
- link field: geometry collision mesh filename=package://field.stl; visual mesh filename=package://field.stl
Joints:
- removed joint field_field_fixed
- removed joint field_goalsally_fixed
- removed joint field_goalsallyback_fixed
- removed joint field_goalsopponent_fixed
- removed joint field_goalsopponentback_fixed
- removed joint field_lines_fixed
- removed joint field_penaltyally_fixed
- removed joint field_penaltyopponent_fixed
- removed joint field_table2_fixed
- removed joint field_table3_fixed
- removed joint field_table4_fixed
- removed joint field_table_fixed
- added joint base_link_to_field: type fixed, parent base_link, child field, origin xyz=0 0 0 rpy=0 -0 0, axis 0 0 1, limit effort=10 velocity=10
- added joint base_link_to_goalsally: type fixed, parent base_link, child goalsally, origin xyz=0 0 0 rpy=0 -0 0, axis 0 0 1, limit effort=10 velocity=10
- added joint base_link_to_goalsallyback: type fixed, parent base_link, child goalsallyback, origin xyz=0 0 0 rpy=0 -0 0, axis 0 0 1, limit effort=10 velocity=10
- added joint base_link_to_goalsopponent: type fixed, parent base_link, child goalsopponent, origin xyz=0 0 0 rpy=0 -0 0, axis 0 0 1, limit effort=10 velocity=10
- added joint base_link_to_goalsopponentback: type fixed, parent base_link, child goalsopponentback, origin xyz=0 0 0 rpy=0 -0 0, axis 0 0 1, limit effort=10 velocity=10
- added joint base_link_to_lines: type fixed, parent base_link, child lines, origin xyz=0 0 0 rpy=0 -0 0, axis 0 0 1, limit effort=10 velocity=10
- added joint base_link_to_penaltyally: type fixed, parent base_link, child penaltyally, origin xyz=0 0 0 rpy=0 -0 0, axis 0 0 1, limit effort=10 velocity=10
- added joint base_link_to_penaltyopponent: type fixed, parent base_link, child penaltyopponent, origin xyz=0 0 0 rpy=0 -0 0, axis 0 0 1, limit effort=10 velocity=10
- added joint base_link_to_table: type fixed, parent base_link, child table, origin xyz=0 0 0 rpy=0 -0 0, axis 0 0 1, limit effort=10 velocity=10
- added joint base_link_to_table2: type fixed, parent base_link, child table2, origin xyz=0 0 0 rpy=0 -0 0, axis 0 0 1, limit effort=10 velocity=10
- added joint base_link_to_table3: type fixed, parent base_link, child table3, origin xyz=0 0 0 rpy=0 -0 0, axis 0 0 1, limit effort=10 velocity=10
- added joint base_link_to_table4: type fixed, parent base_link, child table4, origin xyz=0 0 0 rpy=0 -0 0, axis 0 0 1, limit effort=10 velocity=10

Commit message: Updating field example

File: field_urdf/robot.urdf (robot description, URDF)
Before this commit: robot field_urdf, 13 links, 12 joints
Links:
- link field: geometry collision mesh filename=package://assets/field.stl; visual mesh filename=package://assets/field.stl
- link goalsally: geometry collision mesh filename=package://assets/goalsally.stl; visual mesh filename=package://assets/goalsally.stl
- link goalsallyback: geometry collision mesh filename=package://assets/goalsallyback.stl; visual mesh filename=package://assets/goalsallyback.stl
- link goalsopponent: geometry collision mesh filename=package://assets/goalsopponent.stl; visual mesh filename=package://assets/goalsopponent.stl
- link goalsopponentback: geometry collision mesh filename=package://assets/goalsopponentback.stl; visual mesh filename=package://assets/goalsopponentback.stl
- link lines: geometry collision mesh filename=package://assets/lines.stl; visual mesh filename=package://assets/lines.stl
- link penaltyally: geometry collision mesh filename=package://assets/penaltyally.stl; visual mesh filename=package://assets/penaltyally.stl
- link penaltyopponent: geometry collision mesh filename=package://assets/penaltyopponent.stl; visual mesh filename=package://assets/penaltyopponent.stl
- link table: geometry collision mesh filename=package://assets/table.stl; visual mesh filename=package://assets/table.stl
- link table2: geometry collision mesh filename=package://assets/table2.stl; visual mesh filename=package://assets/table2.stl
- link table3: geometry collision mesh filename=package://assets/table3.stl; visual mesh filename=package://assets/table3.stl
- link table4: geometry collision mesh filename=package://assets/table4.stl; visual mesh filename=package://assets/table4.stl
