Commit message: Updating dog example

File: dog_urdf/robot.urdf (robot description, URDF)
Before this commit: robot dog_urdf, 13 links, 12 joints
Links:
- link body: geometry collision mesh filename=package://assets/merged/body.stl; visual mesh filename=package://assets/merged/body.stl
- link leg_middle: geometry collision mesh filename=package://assets/merged/leg_middle.stl; visual mesh filename=package://assets/merged/leg_middle.stl
- link leg_middle_2: geometry collision mesh filename=package://assets/merged/leg_middle_2.stl; visual mesh filename=package://assets/merged/leg_middle_2.stl
- link leg_middle_3: geometry collision mesh filename=package://assets/merged/leg_middle_3.stl; visual mesh filename=package://assets/merged/leg_middle_3.stl
- link leg_middle_4: geometry collision mesh filename=package://assets/merged/leg_middle_4.stl; visual mesh filename=package://assets/merged/leg_middle_4.stl
- link leg_tip: geometry collision mesh filename=package://assets/merged/leg_tip.stl; visual mesh filename=package://assets/merged/leg_tip.stl
- link leg_tip_2: geometry collision mesh filename=package://assets/merged/leg_tip_2.stl; visual mesh filename=package://assets/merged/leg_tip_2.stl
- link leg_tip_3: geometry collision mesh filename=package://assets/merged/leg_tip_3.stl; visual mesh filename=package://assets/merged/leg_tip_3.stl
- link leg_tip_4: geometry collision mesh filename=package://assets/merged/leg_tip_4.stl; visual mesh filename=package://assets/merged/leg_tip_4.stl
- link leg_top: geometry collision mesh filename=package://assets/merged/leg_top.stl; visual mesh filename=package://assets/merged/leg_top.stl
- link leg_top_2: geometry collision mesh filename=package://assets/merged/leg_top_2.stl; visual mesh filename=package://assets/merged/leg_top_2.stl
- link leg_top_3: geometry collision mesh filename=package://assets/merged/leg_top_3.stl; visual mesh filename=package://assets/merged/leg_top_3.stl
- link leg_top_4: geometry collision mesh filename=package://assets/merged/leg_top_4.stl; visual mesh filename=package://assets/merged/leg_top_4.stl
Joints:
- joint bl_1: origin xyz=0.071 0.3102 0.0234 rpy=-1.5708 7.93087e-13 -3.29157e-13 -> xyz=0.071 0.3102 0.0234 rpy=-1.5708 7.93087e-13 1.25488e-13
- joint bl_3: origin xyz=0.078 -5.55112e-17 -6.93889e-18 rpy=3.14159 -5.55112e-17 -1.5708 -> xyz=0.078 0 0 rpy=3.14159 -5.55112e-17 -1.5708
- joint br_1: origin xyz=-0.028 0.3102 0.0234 rpy=1.5708 -8.05429e-13 3.14159 -> xyz=-0.028 0.3102 0.0234 rpy=1.5708 -8.05429e-13 -3.14159
- joint br_3: origin xyz=0.078 5.55112e-17 0 rpy=3.14159 2.22045e-16 -1.5708 -> xyz=0.078 0 -8.67362e-19 rpy=3.14159 2.22045e-16 -1.5708
- joint fl_1: origin xyz=0.071 0.0398 0.0234 rpy=1.5708 -8.2534e-13 -3.31211e-13 -> xyz=0.071 0.0398 0.0234 rpy=1.5708 -8.25309e-13 1.23434e-13
- joint fl_2: origin xyz=-0.0232 -0.0768608 0.0231 rpy=-1.5708 5.34711e-16 -1.5708 -> xyz=-0.0232 -0.0768608 0.0231 rpy=-1.5708 -1.5827e-15 -1.5708
- joint fl_3: origin xyz=0.078 -2.08167e-17 6.93889e-18 rpy=-3.14159 -6.38378e-16 -1.5708 -> xyz=0.078 -6.93889e-18 6.93889e-18 rpy=-3.14159 -6.38378e-16 -1.5708
- joint fr_1: origin xyz=-0.028 0.0398 0.0231 rpy=-1.5708 7.96373e-13 3.14159 -> xyz=-0.028 0.0398 0.0231 rpy=-1.5708 7.96373e-13 -3.14159
- joint fr_3: origin xyz=0.078 0 0 rpy=3.14159 4.71833e-16 -1.5708 -> xyz=0.078 1.04083e-17 0 rpy=3.14159 4.71833e-16 -1.5708

Commit message: Updating examples

File: dog_urdf/robot.urdf (robot description, URDF)
Before this commit: robot dog_urdf, 13 links, 12 joints
Links:
- link body: geometry collision mesh filename=package://assets/merged/body_collision.stl; visual mesh filename=package://assets/merged/body_visual.stl
- link leg_middle: geometry collision mesh filename=package://assets/merged/leg_middle_collision.stl; visual mesh filename=package://assets/merged/leg_middle_visual.stl
- link leg_middle_2: geometry collision mesh filename=package://assets/merged/leg_middle_2_collision.stl; visual mesh filename=package://assets/merged/leg_middle_2_visual.stl
- link leg_middle_3: geometry collision mesh filename=package://assets/merged/leg_middle_3_collision.stl; visual mesh filename=package://assets/merged/leg_middle_3_visual.stl
- link leg_middle_4: geometry collision mesh filename=package://assets/merged/leg_middle_4_collision.stl; visual mesh filename=package://assets/merged/leg_middle_4_visual.stl
- link leg_tip: geometry collision mesh filename=package://assets/merged/leg_tip_collision.stl; visual mesh filename=package://assets/merged/leg_tip_visual.stl
- link leg_tip_2: geometry collision mesh filename=package://assets/merged/leg_tip_2_collision.stl; visual mesh filename=package://assets/merged/leg_tip_2_visual.stl
- link leg_tip_3: geometry collision mesh filename=package://assets/merged/leg_tip_3_collision.stl; visual mesh filename=package://assets/merged/leg_tip_3_visual.stl
- link leg_tip_4: geometry collision mesh filename=package://assets/merged/leg_tip_4_collision.stl; visual mesh filename=package://assets/merged/leg_tip_4_visual.stl
- link leg_top: geometry collision mesh filename=package://assets/merged/leg_top_collision.stl; visual mesh filename=package://assets/merged/leg_top_visual.stl
- link leg_top_2: geometry collision mesh filename=package://assets/merged/leg_top_2_collision.stl; visual mesh filename=package://assets/merged/leg_top_2_visual.stl
- link leg_top_3: geometry collision mesh filename=package://assets/merged/leg_top_3_collision.stl; visual mesh filename=package://assets/merged/leg_top_3_visual.stl
- link leg_top_4: geometry collision mesh filename=package://assets/merged/leg_top_4_collision.stl; visual mesh filename=package://assets/merged/leg_top_4_visual.stl

File: sigmaban2019_urdf/robot.urdf (robot description, URDF)
Before this commit: robot sigmaban2019_urdf, 27 links, 26 joints
Links:
- link head: geometry collision box size=0.008 0.05 0.003; collision box size=0.008 0.05 0.003
- link left_foot_cleat_front_right: geometry collision box size=0.01 0.09 0.01; collision box size=0.025 0.044 0.003
- link left_humerus: geometry collision box size=0.003 0.07 0.03; collision box size=0.029 0.05 0.04
- link left_knee: geometry collision box size=0.03 0.055 0.04; collision box size=0.04 0.09 0.003
- link left_radius: geometry collision box size=0.003 0.085 0.03; collision box size=0.029 0.05 0.04
- link mx106_block: geometry collision box size=0.03 0.055 0.04; collision box size=0.03 0.055 0.04
- link mx106_block_2: geometry collision box size=0.03 0.055 0.04; collision box size=0.03 0.055 0.04
- link mx106_block_mir: geometry collision box size=0.03 0.055 0.04; collision box size=0.03 0.055 0.04
- link mx106_block_mir_2: geometry collision box size=0.03 0.055 0.04; collision box size=0.03 0.055 0.04
- link right_foot_cleat_back_left: geometry collision box size=0.01 0.09 0.01; collision box size=0.025 0.044 0.003
- link right_humerus: geometry collision box size=0.003 0.07 0.03; collision box size=0.029 0.05 0.04
- link right_knee: geometry collision box size=0.03 0.055 0.04; collision box size=0.04 0.09 0.003
- link right_radius: geometry collision box size=0.003 0.085 0.03; collision box size=0.029 0.05 0.04
- link tibia: geometry collision box size=0.03 0.165 0.003; collision box size=0.03 0.165 0.003
- link tibia_2: geometry collision box size=0.03 0.165 0.003; collision box size=0.03 0.165 0.003
- link tronc: geometry collision box size=0.01 0.035 0.003; collision box size=0.01 0.035 0.003
- link u_block: geometry collision box size=0.025 0.044 0.003; collision box size=0.027 0.042 0.003
- link u_block_2: geometry collision box size=0.025 0.044 0.003; collision box size=0.027 0.042 0.003
- link u_neck: geometry collision box size=0.025 0.044 0.003; collision box size=0.025 0.044 0.003
- link u_shoulder: geometry visual mesh filename=package://assets/merged/u_shoulder_visual.stl
- link u_shoulder_2: geometry visual mesh filename=package://assets/merged/u_shoulder_2_visual.stl
